File: HW/Main/Mini-DSP.kicad_sch (KiCad schematic)
At the start: 98 parts, among them J1 9V, J2 Barrel_Jack_MountingPin, J3 MOBO_Con, J4 SWD, J5 USB_C_Receptacle_USB2.0_16P, SW1 USB_BOOT, SW2 USB_BOOT, SW3 MODE, U2 AMS1117-3.3, U3 W25Q128JVS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

Commit message: test board update
Parts:
- removed C11: 100n, Capacitor_SMD:C_0402_1005Metric, symbol Device:C
- removed C9: 10u, Capacitor_SMD:C_0603_1608Metric, symbol Device:C
- removed J4: SWD, Connector_PinHeader_1.27mm:PinHeader_1x03_P1.27mm_Vertical, symbol Connector:Conn_01x03_Pin
- removed TP2: Vref_aop, TestPoint:TestPoint_Pad_D1.0mm, symbol Connector:TestPoint
- added SW4: ~, AREA_lib_composant:3PDT_LED, symbol AREA_composant:3PDT_Switch
- Audio1, Audio2: footprint easyeda2kicad:AUDIO-TH_PJ-603A -> AREA_lib_composant:AUDIO-TH_PJ-603A_1
- U3: now fitted
- U5: now not fitted
- U6: value RP2354A-QFN60 -> RP2350A
Connections:
- net ~{MUTE_A} is gone; now on an unnamed net: U6.9 (GPIO6)
- net +3V3: now also R4.1
- net +9V: no longer R3.1
- net GND: now also R3.1; no longer R4.2
- net I^{2}S_LRCK: now also U6.15 (GPIO11); no longer U6.14 (GPIO10)
- net I^{2}S_SCLK: now also U6.14 (GPIO10); no longer U6.15 (GPIO11)
- net POT_1: now also U6.42 (GPIO28_ADC2); no longer U6.40 (GPIO26_ADC0)
- net POT_3: now also U6.40 (GPIO26_ADC0); no longer U6.42 (GPIO28_ADC2)
- net SW1: now also U6.35 (GPIO23); no longer U6.3 (GPIO1)
- net SW2: now also U6.34 (GPIO22); no longer U6.4 (GPIO2)
- net at R30.1: no longer U6.32 (GPIO20)
- net Vref_AOP: no longer names the net of R3.2
- net Vref_AOP: now also SW4.2 (A); no longer R4.1
- net ~{MUTE_B}: no longer names the net of U6.10 (GPIO7)
- new net: R4.2, SW4.8 (C)
- new net ON_OFF: SW4.5 (B), U6.32 (GPIO20)
- no-connect marks 4 -> 7
Other:
- moved on the sheet: D3, R30
